Commit message: Fix example models to not depend from laas_objects

File: res/urdf/blue_bin.urdf (robot description, URDF)
Before this commit: robot blue_bin, 1 links, 0 joints
Links:
- link blue_bin: geometry collision box size=0.27 0.36 0.02; collision box size=0.27 0.36 0.02

File: res/urdf/floor.urdf (robot description, URDF)
Before this commit: robot floor, 1 links, 0 joints
Links:
- link floorLink: geometry collision box size=200 200 0.001; visual mesh filename=package://uwds/res/obj/plane.obj scale=1 1 1

File: res/urdf/green_bin.urdf (robot description, URDF)
Before this commit: robot green_bin, 1 links, 0 joints
Links:
- link green_bin: geometry collision box size=0.27 0.36 0.02; collision box size=0.27 0.36 0.02

File: res/urdf/green_cylinder.urdf (robot description, URDF)
Before this commit: robot green_cylinder, 1 links, 0 joints
Links:
- link green_cylinder: geometry collision mesh filename=package://laas_objects/res/obj/green_cylinder.obj; visual mesh filename=package://uwds/res/obj/green_cylinder.obj

File: res/urdf/orange_cup.urdf (robot description, URDF)
Before this commit: robot orange_cup, 1 links, 0 joints
Links:
- link orange_cup: geometry collision mesh filename=package://laas_objects/res/obj/orange_cup.obj; visual mesh filename=package://uwds/res/obj/orange_cup.obj

File: res/urdf/plane.urdf (robot description, URDF)
Before this commit: robot plane, 1 links, 0 joints
Links:
- link planeLink: geometry collision box size=200 200 0.001; visual mesh filename=package://uwds/res/obj/plane.obj scale=1 1 1

File: res/urdf/table.urdf (robot description, URDF)
Before this commit: robot IKEA_table_TORSBY, 1 links, 0 joints
Links:
- link IKEA_table_TORSBY: geometry collision box size=0.025 0.025 0.75; collision box size=0.025 0.025 0.75
