Commit message: Fix example models to not depend from laas_objects

File: res/urdf/green_cylinder.urdf (robot description, URDF)
Before this commit: robot green_cylinder, 1 links, 0 joints
Links:
- link green_cylinder: geometry collision mesh filename=package://uwds/res/obj/green_cylinder.obj; visual mesh filename=package://uwds/res/obj/green_cylinder.obj

File: res/urdf/orange_cup.urdf (robot description, URDF)
Before this commit: robot orange_cup, 1 links, 0 joints
Links:
- link orange_cup: geometry collision mesh filename=package://uwds/res/obj/orange_cup.obj; visual mesh filename=package://uwds/res/obj/orange_cup.obj
